File: KiCad/RaspPi.kicad_sch (KiCad schematic)
At the start: 9 parts, among them J101 Raspberry_Pi_2_3

Commit message: Schaltplan Update
Parts:
- added RCWL-I2CAdapter: ~, symbol 0wörk_sym:BNO080
Connections:
- net SCL2: no longer R101.1
- net SDA2: no longer R102.1
- net at J101.31 (GCLK2/GPIO6): no longer RCWL-0516. (VCC)
- net at J101.3 (SDA1/GPIO2): now also R102.1
- net at J101.5 (SCL1/GPIO3): now also R101.1
- new net: RCWL-0516. (VCC), RCWL-I2CAdapter. (VCC) (x2)
- new net SCL6: RCWL-I2CAdapter. (VCC)
- new net SDA6: RCWL-I2CAdapter. (VCC)
- no-connect marks 1 -> 0
Other:
- note added: "I2C Adress: 0x25 Für SDP610: 64 (1000000)"
- note added: "I2C Adress: 0x49/48/4A/4B"
- note removed: "I2C Adress: 0x25 Für SDP610: 64 (1000000) Pull-Ups (10k) on SDA & SCL"
- moved on the sheet: J101, R101, R102, RCWL-0516
